File: hardware/max31856.kicad_sch (KiCad schematic)
At the start: 14 parts, among them U4 MAX31856

Commit message: chore(hw): migrate KiCad files to the KiCad 10 format
Via `kicad-cli sch upgrade` / `pcb upgrade` (bread-infra
scripts/upgrade_kicad10.sh). Verified lossless: identical netlist, footprint
positions and routing.

Note `sch upgrade` does not cascade into hierarchical sub-sheets, so every
.kicad_sch is upgraded individually -- upgrading only the root sheet leaves
sub-sheets on the old format, which looks migrated and is not.
Parts:
- renumbered C7 to C17, C8 to C18, C9 to C19, C10 to C20, C11 to C21, D4 to D10, D2 to D8, D3 to D9, R1 to R11, R2 to R12, R3 to R13, R4 to R14, R5 to R15, U4 to U6
