File: hardware/BREAD_Slice.kicad_pcb (KiCad board)
At the start: 2 copper layers, 70 x 100 mm, 83 parts, among them J1 I2C_01x04, J2 Conn_01x10_Female, J4 Conn_01x02, J5 Conn_01x02, J6 Conn_01x02, J7 Conn_01x02, U2 CD74HC4053E, U3 MIC5225-3.3YM5-TR, U4 MAX31856, U5 MAX31856, U6 MAX31856, U7 MAX31856

Commit message: fix(hw): re-point stale library nicknames
These parts exist in KiCad-Master-Lib; the boards referenced libraries that no
longer exist (kml-custom, KML-Custom, and SparkFun libraries that never
contained the part) or names the library has since changed.

KiCad embeds footprint geometry in the .kicad_pcb, so the boards rendered and
fabricated correctly and the rot stayed invisible -- it only surfaces on
update-from-library, or when a generator tries to resolve a nickname.

Nickname/name only. No geometry is changed:

  KML-Custom:DIP254P762X508-16 -> KMLib_IC_THT:DIP254P762X508-16
  KML-Custom:Thermal Pad -> KMLib_Mounting:Thermal_Pad
  SparkFun-DiscreteSemi:AP63205 -> KMLib_IC_Power:AP63205WU-7_Buck_Regulator
  SparkFun-LED:WS2812-5050-4PIN -> KMLib_IC_SMD:WS2812-5050-4PIN
  kml-custom:CD74HC4053E -> KMLib_IC_Analog:CD74HC4053E_Multiplexer

Only references that failed to resolve were touched. Generic parts (<=4 pins)
and KiCad *-rescue libraries are deliberately excluded: fingerprint matching
cannot distinguish a 2-pin resistor from a 2-pin capacitor, so those are being
done by hand.
Parts:
- D1: footprint SparkFun-LED:WS2812-5050-4PIN -> KMLib_IC_SMD:WS2812-5050-4PIN
- HS1: footprint KML-Custom:Thermal Pad -> KMLib_Mounting:Thermal_Pad
- U2: footprint KML-Custom:DIP254P762X508-16 -> KMLib_IC_THT:DIP254P762X508-16
Changed lines of the file:
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@@
 		)
 	)
-	(footprint "KML-Custom:Thermal Pad"
+	(footprint "KMLib_Mounting:Thermal_Pad"
 		(layer "F.Cu")
 		(at 135.3 62.7)
@@
 		(embedded_fonts no)
 	)
-	(footprint "SparkFun-LED:WS2812-5050-4PIN"
+	(footprint "KMLib_IC_SMD:WS2812-5050-4PIN"
 		(locked yes)
 		(layer "F.Cu")
@@
 		(embedded_fonts no)
 	)
-	(footprint "KML-Custom:DIP254P762X508-16"
+	(footprint "KMLib_IC_THT:DIP254P762X508-16"
 		(layer "F.Cu")
 		(at 160.26 131.71 -90)
